File: hardware/prj-kicad/cowmod.sch (KiCad schematic (older format))
At the start: 0 parts

Commit message: = ADD: Insert FPGA and route all PMOD ports
Parts:
- added P1, P2, P3, P4: PMOD, cowmod:PMOD_SSW106-RA, symbol PMOD
Connections:
- new net +PMOD1: P1.12, P1.6
- new net +PMOD2: P2.12, P2.6
- new net +PMOD3: P3.12, P3.6
- new net +PMOD4: P4.12, P4.6
- new net GND: P1.11, P1.5, P2.11, P2.5, P3.11, P3.5, P4.11, P4.5
- new net P1_IO1: P1.1 (IO1)
- new net P1_IO2: P1.2 (IO2)
- new net P1_IO3: P1.3 (IO3)
- new net P1_IO4: P1.4 (IO4)
- new net P1_IO5: P1.7 (IO5)
- new net P1_IO6: P1.8 (IO6)
- new net P1_IO7: P1.9 (IO7)
- new net P1_IO8: P1.10 (IO8)
- new net P2_IO1: P2.1 (IO1)
- new net P2_IO2: P2.2 (IO2)
- new net P2_IO3: P2.3 (IO3)
- new net P2_IO4: P2.4 (IO4)
- new net P2_IO5: P2.7 (IO5)
- new net P2_IO6: P2.8 (IO6)
- new net P2_IO7: P2.9 (IO7)
- new net P2_IO8: P2.10 (IO8)
- new net P3_IO1: P3.1 (IO1)
- new net P3_IO2: P3.2 (IO2)
- new net P3_IO3: P3.3 (IO3)
- new net P3_IO4: P3.4 (IO4)
- new net P3_IO5: P3.7 (IO5)
- new net P3_IO6: P3.8 (IO6)
- new net P3_IO7: P3.9 (IO7)
- new net P3_IO8: P3.10 (IO8)
- new net P4_IO1: P4.1 (IO1)
- new net P4_IO2: P4.2 (IO2)
- new net P4_IO3: P4.3 (IO3)
- new net P4_IO4: P4.4 (IO4)
- new net P4_IO5: P4.7 (IO5)
- new net P4_IO6: P4.8 (IO6)
- new net P4_IO7: P4.9 (IO7)
- new net P4_IO8: P4.10 (IO8)

Commit message: = ADD: Insert main MCU (STM32) and connect it to FPGA
Changed lines of the file:
@@
 $Descr A4 11693 8268
 encoding utf-8
-Sheet 1 3
+Sheet 1 4
 Title "Cowmod 4MVII"
 Date "2019-05-29"
@@
 F1 "cowmod-fpga.sch" 60
 $EndSheet
+$Sheet
+S 3600 1650 2500 1400
+U 5CF5FBFC
+F0 "MCU" 60
+F1 "cowmod-mcu.sch" 60
+$EndSheet
 $EndSCHEMATC
